File: hw/kicad/v1/v1.kicad_pcb (KiCad board)
At the start: 4 copper layers, 100 x 100 mm, 146 parts, among them J101 Conn_01x03_Pin, J102 031-6575, J201 Screw_Terminal_01x04, J202 Screw_Terminal_01x03, J601 Conn_01x04_Pin, J602 Conn_01x16_Pin, J603 USB_C_Receptacle_USB2.0_16P, SW601 SW_MEC_5E, SW602 SW_MEC_5E, U1001 4051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

Commit message: production gerber files
Parts:
- moved H101 1.41 mm to (45.0, 65.0)
- moved H102 1.41 mm to (45.0, 155.0)
Routing:
- net GND: track 14.0 -> 20.0 mm, vias 274 -> 275
Changed lines of the file:
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@@
 		(tags "capacitor handsolder")
 		(property "Reference" "C1003"
-			(at 0 -1.85 0)
+			(at 5.3 -0.1 0)
 			(layer "F.SilkS")
 			(effects
@@
 			(at 0 -3.8 0)
 			(layer "F.SilkS")
+			(hide yes)
 			(effects
 				(font
@@
 		(tags "capacitor handsolder")
 		(property "Reference" "C203"
-			(at -0.0375 2.2 0)
+			(at 5.1625 0 0)
 			(layer "F.SilkS")
 			(effects
@@
 		(tags "Through hole pin header THT 1x04 2.54mm single row")
 		(property "Reference" "J601"
-			(at 0 -10.32 0)
+			(at -0.5 -2.6 0)
 			(layer "F.SilkS")
 			(effects
@@
 	(footprint "MountingHole:MountingHole_3.2mm_M3_ISO7380_Pad_TopBottom"
 		(layer "F.Cu")
-		(at 46 154)
+		(at 45 155)
 		(descr "Mounting Hole 3.2mm, M3, generated by kicad-footprint-generator mountinghole.py")
 		(tags "mountinghole M3 ISO7380")
@@
 			(at 0 -3.8 0)
 			(layer "F.SilkS")
+			(hide yes)
 			(effects
 				(font
@@
 	(footprint "MountingHole:MountingHole_3.2mm_M3_ISO7380_Pad_TopBottom"
 		(layer "F.Cu")
-		(at 46 66)
+		(at 45 65)
 		(descr "Mounting Hole 3.2mm, M3, generated by kicad-footprint-generator mountinghole.py")
 		(tags "mountinghole M3 ISO7380")
@@
 			(at 0 -3.8 0)
 			(layer "F.SilkS")
+			(hide yes)
 			(effects
 				(font
@@
 			(at -5.4 2 0)
 			(layer "F.SilkS")
+			(hide yes)
 			(effects
 				(font
@@
 		(tags "THT terminal block MaiXu MX126-5.0-04P pitch 5mm size 20.5x7.8mm drill 1.3mm pad 2.8mm")
 		(property "Reference" "J201"
-			(at 7.25 -5.12 90)
+			(at 5.2 4.8 90)
 			(layer "F.SilkS")
 			(effects
@@
 		(layer "Dwgs.User")
 		(pts
-			(xy 46 66) (xy 135 66)
+			(xy 45 66) (xy 135 65)
 		)
 		(height -25.4)
@@
 			(keep_text_aligned yes)
 		)
-		(gr_text "89"
-			(at 90.5 39.45 0)
+		(gr_text "90"
+			(at 90 39.45 0)
 			(layer "Dwgs.User")
 			(effects
@@
 	)
 	(segment
+		(start 54.6 96.1)
+		(end 54.2 96.5)
+		(width 0.2)
+		(layer "F.Cu")
+		(net 1)
+	)
+	(segment
+		(start 54.2 96.5)
+		(end 53.6 96.5)
+		(width 0.2)
+		(layer "F.Cu")
+		(net 1)
+	)
+	(segment
 		(start 61.55 123.1)
 		(end 62.1 123.1)
@@
 	)
 	(segment
+		(start 55.45 96.1)
+		(end 54.6 96.1)
+		(width 0.2)
+		(layer "F.Cu")
+		(net 1)
+	)
+	(segment
 		(start 94.381061 148.418939)
 		(end 94.505 148.295)
@@
 	)
 	(segment
+		(start 113.8 130.4)
+		(end 112.8 131.4)
+		(width 0.2)
+		(layer "F.Cu")
+		(net 1)
+	)
+	(segment
 		(start 60.9 123.1)
 		(end 61.55 123.1)
@@
 	)
 	(segment
+		(start 55.45 96.1)
+		(end 56.8 96.1)
+		(width 0.2)
+		(layer "F.Cu")
+		(net 1)
+	)
+	(segment
 		(start 60.7 70.62)
 		(end 60.7 69.32)
@@
 	)
 	(segment
+		(start 113.8 129.2)
+		(end 113.8 130.4)
+		(width 0.2)
+		(layer "F.Cu")
+		(net 1)
+	)
+	(segment
 		(start 58.5 123.4375)
 		(end 57.2375 123.4375)
@@
 	)
 	(via
-		(at 70 73.99)
+		(at 70 74.4)
 		(size 0.6)
 		(drill 0.3)
@@
 	)
 	(via
+		(at 116.3 136.5)
+		(size 0.6)
+		(drill 0.3)
+		(layers "F.Cu" "B.Cu")
+		(free yes)
+		(net 1)
+	)
+	(via
 		(at 63.1 90.7)
 		(size 0.6)
@@
 	)
 	(via
-		(at 74 73.99)
+		(at 74 74.4)
 		(size 0.6)
 		(drill 0.3)
@@
 	)
 	(via
-		(at 98 73.99)
+		(at 98 74.4)
 		(size 0.6)
 		(drill 0.3)
@@
 	)
 	(via
-		(at 90 73.99)
+		(at 90 74.4)
 		(size 0.6)
 		(drill 0.3)
@@
 	)
 	(via
-		(at 51.3 92.3)
+		(at 51.1 92.1)
 		(size 0.6)
 		(drill 0.3)
@@
 	)
 	(via
-		(at 66 73.99)
+		(at 66 74.4)
 		(size 0.6)
 		(drill 0.3)
@@
 	)
 	(via
-		(at 94 73.99)
+		(at 94 74.4)
 		(size 0.6)
 		(drill 0.3)
@@
 	)
 	(via
-		(at 86 73.99)
+		(at 86 74.4)
 		(size 0.6)
 		(drill 0.3)
@@
 	)
 	(via
-		(at 82 73.99)
+		(at 82 74.4)
 		(size 0.6)
 		(drill 0.3)
@@
 	)
 	(via
-		(at 78 73.99)
+		(at 78 74.4)
 		(size 0.6)
 		(drill 0.3)
@@
 	)
 	(via
-		(at 115.8 131.4)
+		(at 116.3 131.4)
 		(size 0.6)
 		(drill 0.3)
@@
 	)
 	(segment
-		(start 114.2375 127.3)
-		(end 114.2375 126.9)
+		(start 115.2 128.1)
+		(end 115.2 128.7)
 		(width 0.5)
 		(layer "F.Cu")
@@
 	)
 	(segment
-		(start 114.7 128.5)
-		(end 114.7 127.7625)
-		(width 0.5)
+		(start 111.3375 135.0625)
+		(end 111.3375 136.5)
+		(width 0.2)
 		(layer "F.Cu")
 		(net 15)
 	)
 	(segment
-		(start 111.3375 135.0625)
-		(end 111.3375 136.5)
-		(width 0.2)
+		(start 114.2375 127.1375)
+		(end 115.2 128.1)
+		(width 0.5)
 		(layer "F.Cu")
 		(net 15)
@@
 	)
 	(segment
-		(start 114.7 127.7625)
-		(end 114.2375 127.3)
-		(width 0.5)
-		(layer "F.Cu")
-		(net 15)
-	)
-	(segment
 		(start 111.8 133.6)
 		(end 111.8 134.6)
@@
 	)
 	(segment
+		(start 114.2375 126.9)
+		(end 114.2375 127.1375)
+		(width 0.5)
+		(layer "F.Cu")
+		(net 15)
+	)
+	(segment
 		(start 113.8375 127.3)
 		(end 114.2375 126.9)
@@
 	)
 	(via
-		(at 114.7 128.5)
+		(at 115.2 128.7)
 		(size 0.6)
 		(drill 0.3)
@@
 	)
 	(segment
-		(start 52.2 96.5)
-		(end 43.6 105.1)
+		(start 111.8 139.3)
+		(end 115.2 135.9)
 		(width 0.5)
 		(layer "In2.Cu")
@@
 	)
 	(segment
-		(start 55.9885 142.951)
-		(end 110.149 142.951)
+		(start 52.2 96.5)
+		(end 43.6 105.1)
 		(width 0.5)
 		(layer "In2.Cu")
@@
 	)
 	(segment
-		(start 111.8 139.3)
-		(end 114.7 136.4)
+		(start 115.2 135.9)
+		(end 115.2 128.7)
 		(width 0.5)
 		(layer "In2.Cu")
@@
 	)
 	(segment
-		(start 53.887499 140.849999)
-		(end 55.9885 142.951)
+		(start 55.9885 142.951)
+		(end 110.149 142.951)
 		(width 0.5)
 		(layer "In2.Cu")
@@
 	)
 	(segment
-		(start 114.7 136.4)
-		(end 114.7 128.5)
+		(start 53.887499 140.849999)
+		(end 55.9885 142.951)
 		(width 0.5)
 		(layer "In2.Cu")
@@
 	)
 	(segment
-		(start 106.8 76.695)
-		(end 98.995 76.695)
+		(start 63.63 75.3)
+		(end 61.65 73.32)
 		(width 0.2)
 		(layer "F.Cu")
@@
 	)
 	(segment
-		(start 98.995 76.695)
-		(end 96.9 74.6)
+		(start 106.8 76.695)
+		(end 98.995 76.695)
 		(width 0.2)
 		(layer "F.Cu")
@@
 	)
 	(segment
-		(start 96.9 74.6)
-		(end 62.93 74.6)
+		(start 97.6 75.3)
+		(end 63.63 75.3)
 		(width 0.2)
 		(layer "F.Cu")
@@
 	)
 	(segment
-		(start 62.93 74.6)
-		(end 61.65 73.32)
+		(start 98.995 76.695)
+		(end 97.6 75.3)
 		(width 0.2)
 		(layer "F.Cu")
@@
 	)
 	(segment
-		(start 96.08179 75.4)
+		(start 96.48179 75.8)
 		(end 98.64679 77.965)
 		(width 0.2)
@@
 	(segment
 		(start 59.75 75.15)
-		(end 60 75.4)
+		(end 60.4 75.8)
 		(width 0.2)
 		(layer "F.Cu")
@@
 	)
 	(segment
-		(start 98.64679 77.965)
-		(end 106.8 77.965)
+		(start 59.75 73.32)
+		(end 59.75 75.15)
 		(width 0.2)
 		(layer "F.Cu")
@@
 	)
 	(segment
-		(start 59.75 73.32)
-		(end 59.75 75.15)
+		(start 60.4 75.8)
+		(end 96.48179 75.8)
 		(width 0.2)
 		(layer "F.Cu")
@@
 	)
 	(segment
-		(start 60 75.4)
-		(end 96.08179 75.4)
+		(start 98.64679 77.965)
+		(end 106.8 77.965)
 		(width 0.2)
 		(layer "F.Cu")
