File: hw/kicad/v1/v1_frontpanel/v1_frontpanel.kicad_pcb (KiCad board)
At the start: 2 copper layers, 100 x 60 mm, 20 parts, among them J101 Conn_01x16_Pin, SW101 SW_Push, SW102 SW_Push, SW103 RotaryEncoder, U101 CR2013-MI2120

Commit message: production gerber files
Changed lines of the file:
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@@
 			(at -0.043742 -6 180)
 			(layer "F.SilkS")
+			(hide yes)
 			(effects
 				(font
@@
 			(at 2 -6 180)
 			(layer "F.SilkS")
+			(hide yes)
 			(effects
 				(font
@@
 			(at -0.2 5.6 180)
 			(layer "F.SilkS")
+			(hide yes)
 			(effects
 				(font
@@
 			(at 4 0 180)
 			(layer "F.SilkS")
-			(effects
-				(font
+			(hide yes)
+			(effects
+				(font
